Commit message: Multicopter Velocity Plugin Resolved - Communication works

File: src/sar_drone_description/urdf/sar_drone.urdf.xacro (robot description, xacro)
@@ -11,4 +11,7 @@
         <cylinder radius="0.2" length="0.1"/>
       </geometry>
+      <material name="drone_body">
+        <color rgba="0.2 0.2 0.2 1.0"/>
+      </material>
     </visual>
     <collision>
@@ -18,4 +21,89 @@
     </collision>
   </link>
+  <!-- ================= ROTORS ================= -->
+  <!-- Front Right Motor (Motor 0) -->
+  <link name="rotor_0">
+    <inertial>
+      <mass value="0.01"/>
+      <inertia ixx="0.0001" ixy="0" ixz="0" iyy="0.0001" iyz="0" izz="0.0001"/>
+    </inertial>
+    <visual>
+      <geometry>
+        <cylinder radius="0.05" length="0.01"/>
+      </geometry>
+      <material name="rotor">
+        <color rgba="0.8 0.1 0.1 1.0"/>
+      </material>
+    </visual>
+  </link>
+  <joint name="rotor_0_joint" type="continuous">
+    <parent link="base_link"/>
+    <child link="rotor_0"/>
+    <origin xyz="0.13 0.13 0.05" rpy="0 0 0"/>
+    <axis xyz="0 0 1"/>
+  </joint>
+  <!-- Front Left Motor (Motor 1) -->
+  <link name="rotor_1">
+    <inertial>
+      <mass value="0.01"/>
+      <inertia ixx="0.0001" ixy="0" ixz="0" iyy="0.0001" iyz="0" izz="0.0001"/>
+    </inertial>
+    <visual>
+      <geometry>
+        <cylinder radius="0.05" length="0.01"/>
+      </geometry>
+      <material name="rotor">
+        <color rgba="0.8 0.1 0.1 1.0"/>
+      </material>
+    </visual>
+  </link>
+  <joint name="rotor_1_joint" type="continuous">
+    <parent link="base_link"/>
+    <child link="rotor_1"/>
+    <origin xyz="-0.13 0.13 0.05" rpy="0 0 0"/>
+    <axis xyz="0 0 1"/>
+  </joint>
+  <!-- Rear Left Motor (Motor 2) -->
+  <link name="rotor_2">
+    <inertial>
+      <mass value="0.01"/>
+      <inertia ixx="0.0001" ixy="0" ixz="0" iyy="0.0001" iyz="0" izz="0.0001"/>
+    </inertial>
+    <visual>
+      <geometry>
+        <cylinder radius="0.05" length="0.01"/>
+      </geometry>
+      <material name="rotor">
+        <color rgba="0.8 0.1 0.1 1.0"/>
+      </material>
+    </visual>
+  </link>
+  <joint name="rotor_2_joint" type="continuous">
+    <parent link="base_link"/>
+    <child link="rotor_2"/>
+    <origin xyz="-0.13 -0.13 0.05" rpy="0 0 0"/>
+    <axis xyz="0 0 1"/>
+  </joint>
+  <!-- Rear Right Motor (Motor 3) -->
+  <link name="rotor_3">
+    <inertial>
+      <mass value="0.01"/>
+      <inertia ixx="0.0001" ixy="0" ixz="0" iyy="0.0001" iyz="0" izz="0.0001"/>
+    </inertial>
+    <visual>
+      <geometry>
+        <cylinder radius="0.05" length="0.01"/>
+      </geometry>
+      <material name="rotor">
+        <color rgba="0.8 0.1 0.1 1.0"/>
+      </material>
+    </visual>
+  </link>
+  <joint name="rotor_3_joint" type="continuous">
+    <parent link="base_link"/>
+    <child link="rotor_3"/>
+    <origin xyz="0.13 -0.13 0.05" rpy="0 0 0"/>
+    <axis xyz="0 0 1"/>
+  </joint>
   <!-- ================= LIDAR ================= -->
   <link name="lidar_link"/>
@@ -83,76 +171,179 @@
     </sensor>
   </gazebo>
-	<!-- IMU -->
-	<gazebo reference="imu_link">
-	  <sensor name="imu" type="imu">
-	    <frame>imu_link</frame>
-	    <topic>/imu/data</topic>
-	    <update_rate>100</update_rate>
-	    <imu>
-	      <angular_velocity>
-		<x>
-		  <noise type="gaussian">
-		    <mean>0.0</mean>
-		    <stddev>0.0002</stddev>
-		    <bias_mean>0.0</bias_mean>
-		    <bias_stddev>0.0001</bias_stddev>
-		  </noise>
-		</x>
-		<y>
-		  <noise type="gaussian">
-		    <mean>0.0</mean>
-		    <stddev>0.0002</stddev>
-		    <bias_mean>0.0</bias_mean>
-		    <bias_stddev>0.0001</bias_stddev>
-		  </noise>
-		</y>
-		<z>
-		  <noise type="gaussian">
-		    <mean>0.0</mean>
-		    <stddev>0.0002</stddev>
-		    <bias_mean>0.0</bias_mean>
-		    <bias_stddev>0.0001</bias_stddev>
-		  </noise>
-		</z>
-	      </angular_velocity>
-	      <linear_acceleration>
-		<x>
-		  <noise type="gaussian">
-		    <mean>0.0</mean>
-		    <stddev>0.017</stddev>
-		    <bias_mean>0.0</bias_mean>
-		    <bias_stddev>0.008</bias_stddev>
-		  </noise>
-		</x>
-		<y>
-		  <noise type="gaussian">
-		    <mean>0.0</mean>
-		    <stddev>0.017</stddev>
-		    <bias_mean>0.0</bias_mean>
-		    <bias_stddev>0.008</bias_stddev>
-		  </noise>
-		</y>
-		<z>
-		  <noise type="gaussian">
-		    <mean>0.0</mean>
-		    <stddev>0.017</stddev>
-		    <bias_mean>0.0</bias_mean>
-		    <bias_stddev>0.008</bias_stddev>
-		  </noise>
-		</z>
-	      </linear_acceleration>
-	    </imu>
-	  </sensor>
-	</gazebo>
-  <!-- ================= SIMPLE VELOCITY CONTROLLER ================= -->
+  <!-- IMU -->
+  <gazebo reference="imu_link">
+    <sensor name="imu" type="imu">
+      <frame>imu_link</frame>
+      <topic>/imu/data</topic>
+      <update_rate>100</update_rate>
+      <imu>
+        <angular_velocity>
+          <x>
+            <noise type="gaussian">
+              <mean>0.0</mean>
+              <stddev>0.0002</stddev>
+              <bias_mean>0.0</bias_mean>
+              <bias_stddev>0.0001</bias_stddev>
+            </noise>
+          </x>
+          <y>
+            <noise type="gaussian">
+              <mean>0.0</mean>
+              <stddev>0.0002</stddev>
+              <bias_mean>0.0</bias_mean>
+              <bias_stddev>0.0001</bias_stddev>
+            </noise>
+          </y>
+          <z>
+            <noise type="gaussian">
+              <mean>0.0</mean>
+              <stddev>0.0002</stddev>
+              <bias_mean>0.0</bias_mean>
+              <bias_stddev>0.0001</bias_stddev>
+            </noise>
+          </z>
+        </angular_velocity>
+        <linear_acceleration>
+          <x>
+            <noise type="gaussian">
+              <mean>0.0</mean>
+              <stddev>0.017</stddev>
+              <bias_mean>0.0</bias_mean>
+              <bias_stddev>0.008</bias_stddev>
+            </noise>
+          </x>
+          <y>
+            <noise type="gaussian">
+              <mean>0.0</mean>
+              <stddev>0.017</stddev>
+              <bias_mean>0.0</bias_mean>
+              <bias_stddev>0.008</bias_stddev>
+            </noise>
+          </y>
+          <z>
+            <noise type="gaussian">
+              <mean>0.0</mean>
+              <stddev>0.017</stddev>
+              <bias_mean>0.0</bias_mean>
+              <bias_stddev>0.008</bias_stddev>
+            </noise>
+          </z>
+        </linear_acceleration>
+      </imu>
+    </sensor>
+  </gazebo>
+  <!-- ================= MULTICOPTER FLIGHT CONTROLLER ================= -->
   <gazebo>
-    <plugin filename="gz-sim-velocity-control-system"
-            name="gz::sim::systems::VelocityControl">
-      <initial_linear>0 0 0</initial_linear>
-      <initial_angular>0 0 0</initial_angular>
-    </plugin>
-    <plugin filename="gz-sim-apply-link-wrench-system"
-            name="gz::sim::systems::ApplyLinkWrench">
-      <link_name>base_link</link_name>
+    <!-- Motor 0: Front Right (CCW) -->
+    <plugin filename="gz-sim-multicopter-motor-model-system"
+            name="gz::sim::systems::MulticopterMotorModel">
+      <jointName>rotor_0_joint</jointName>
+      <linkName>rotor_0</linkName>
+      <turningDirection>ccw</turningDirection>
+      <timeConstantUp>0.0125</timeConstantUp>
+      <timeConstantDown>0.025</timeConstantDown>
+      <maxRotVelocity>1100</maxRotVelocity>
+      <motorConstant>8.54858e-06</motorConstant>
+      <momentConstant>0.06</momentConstant>
+      <commandSubTopic>/gazebo/command/motor_speed</commandSubTopic>
+      <motorNumber>0</motorNumber>
+      <rotorDragCoefficient>0.000806428</rotorDragCoefficient>
+      <rollingMomentCoefficient>1e-06</rollingMomentCoefficient>
+      <rotorVelocitySlowdownSim>10</rotorVelocitySlowdownSim>
+    </plugin>
+    <!-- Motor 1: Front Left (CW) -->
+    <plugin filename="gz-sim-multicopter-motor-model-system"
+            name="gz::sim::systems::MulticopterMotorModel">
+      <jointName>rotor_1_joint</jointName>
+      <linkName>rotor_1</linkName>
+      <turningDirection>cw</turningDirection>
+      <timeConstantUp>0.0125</timeConstantUp>
+      <timeConstantDown>0.025</timeConstantDown>
+      <maxRotVelocity>1100</maxRotVelocity>
+      <motorConstant>8.54858e-06</motorConstant>
+      <momentConstant>0.06</momentConstant>
+      <commandSubTopic>/gazebo/command/motor_speed</commandSubTopic>
+      <motorNumber>1</motorNumber>
+      <rotorDragCoefficient>0.000806428</rotorDragCoefficient>
+      <rollingMomentCoefficient>1e-06</rollingMomentCoefficient>
+      <rotorVelocitySlowdownSim>10</rotorVelocitySlowdownSim>
+    </plugin>
+    <!-- Motor 2: Rear Left (CCW) -->
+    <plugin filename="gz-sim-multicopter-motor-model-system"
+            name="gz::sim::systems::MulticopterMotorModel">
+      <jointName>rotor_2_joint</jointName>
+      <linkName>rotor_2</linkName>
+      <turningDirection>ccw</turningDirection>
+      <timeConstantUp>0.0125</timeConstantUp>
+      <timeConstantDown>0.025</timeConstantDown>
+      <maxRotVelocity>1100</maxRotVelocity>
+      <motorConstant>8.54858e-06</motorConstant>
+      <momentConstant>0.06</momentConstant>
+      <commandSubTopic>/gazebo/command/motor_speed</commandSubTopic>
+      <motorNumber>2</motorNumber>
+      <rotorDragCoefficient>0.000806428</rotorDragCoefficient>
+      <rollingMomentCoefficient>1e-06</rollingMomentCoefficient>
+      <rotorVelocitySlowdownSim>10</rotorVelocitySlowdownSim>
+    </plugin>
+    <!-- Motor 3: Rear Right (CW) -->
+    <plugin filename="gz-sim-multicopter-motor-model-system"
+            name="gz::sim::systems::MulticopterMotorModel">
+      <jointName>rotor_3_joint</jointName>
+      <linkName>rotor_3</linkName>
+      <turningDirection>cw</turningDirection>
+      <timeConstantUp>0.0125</timeConstantUp>
+      <timeConstantDown>0.025</timeConstantDown>
+      <maxRotVelocity>1100</maxRotVelocity>
+      <motorConstant>8.54858e-06</motorConstant>
+      <momentConstant>0.06</momentConstant>
+      <commandSubTopic>/gazebo/command/motor_speed</commandSubTopic>
+      <motorNumber>3</motorNumber>
+      <rotorDragCoefficient>0.000806428</rotorDragCoefficient>
+      <rollingMomentCoefficient>1e-06</rollingMomentCoefficient>
+      <rotorVelocitySlowdownSim>10</rotorVelocitySlowdownSim>
+    </plugin>
+    <!-- Multicopter Velocity Controller -->
+    <plugin filename="gz-sim-multicopter-control-system"
+            name="gz::sim::systems::MulticopterVelocityControl">
+      <robotNamespace>sar_drone</robotNamespace>  ← ADD THIS LINE!
+      <commandSubTopic>cmd_vel</commandSubTopic>
+      <motorControlPubTopic>/gazebo/command/motor_speed</motorControlPubTopic>
+      <enableSubTopic>enable</enableSubTopic>
+      <comLinkName>base_link</comLinkName>
+      <velocityGain>2.7 2.7 5.0</velocityGain>
+      <attitudeGain>4.0 4.0 0.6</attitudeGain>
+      <angularRateGain>0.5 0.5 0.3</angularRateGain>
+      <maximumLinearAcceleration>2.0 2.0 4.0</maximumLinearAcceleration>
+      <maximumAngularVelocity>3.0 3.0 2.0</maximumAngularVelocity>
+      <linearVelocityNoiseMean>0 0 0</linearVelocityNoiseMean>
+      <linearVelocityNoiseStdDev>0.05 0.05 0.05</linearVelocityNoiseStdDev>
+      <angularVelocityNoiseMean>0 0 0</angularVelocityNoiseMean>
+      <angularVelocityNoiseStdDev>0.01 0.01 0.01</angularVelocityNoiseStdDev>
+      <rotorConfiguration>
+        <rotor>
+          <jointName>rotor_0_joint</jointName>
+          <forceConstant>8.54858e-06</forceConstant>
+          <momentConstant>0.06</momentConstant>
+          <direction>1</direction>
+        </rotor>
+        <rotor>
+          <jointName>rotor_1_joint</jointName>
+          <forceConstant>8.54858e-06</forceConstant>
+          <momentConstant>0.06</momentConstant>
+          <direction>-1</direction>
+        </rotor>
+        <rotor>
+          <jointName>rotor_2_joint</jointName>
+          <forceConstant>8.54858e-06</forceConstant>
+          <momentConstant>0.06</momentConstant>
+          <direction>1</direction>
+        </rotor>
+        <rotor>
+          <jointName>rotor_3_joint</jointName>
+          <forceConstant>8.54858e-06</forceConstant>
+          <momentConstant>0.06</momentConstant>
+          <direction>-1</direction>
+        </rotor>
+      </rotorConfiguration>
     </plugin>
   </gazebo>
